File: ecu-board/relays.sch (KiCad schematic (older format))
At the start: 4 parts, among them K1 Main power relay, K2 Start motor relay

Commit message: Rename board signals.
Connections:
- net start_motor_relay_input renamed ~start_motor_relay_input~
Changed lines of the file:
@@
 	1    0    0    -1
 $EndComp
-Text HLabel 6500 3400 0    50   Input ~ 0
-start_motor_relay_input
 Text Notes 2700 2650 0    79   ~ 16
 Main power relay
@@
 Wire Wire Line
 	3950 2950 4250 2950
+Text HLabel 6500 3400 0    50   Input ~ 0
+~start_motor_relay_input~
 $EndSCHEMATC
